File: dronehopefully.kicad_pcb (KiCad board)
At the start: 2 copper layers, 2 x 7.5 mm, 60 parts, among them J1 SBUS, J14 US3TX, J15 US3RX, J16 U4TX, J17 U4RX, J18 U5TX, J19 U5RX, J2 PPM, J20 LED, J5 USB_B_Micro, J6 S1, J7 S2, J8 S3, J9 S4, Q1 BC817W, SW1 SW_SPST, U1 STM32F405RGTx, U2 MIC5319-3.3YD5-TR, U3 MPU-6500, X1 8MHz

Commit message: Add files via upload
Parts:
- removed R2, R3: 10k, Resistor_SMD:R_0402_1005Metric
- R1, R7, R8: moved to B.Cu
- moved R5 4.01 mm to (158.2, 99.5)
- moved R4 3.76 mm to (158.2, 98.2)
- moved R12 3.04 mm to (154.5, 108.5)
- moved C9 2.93 mm to (151.0, 89.0)
- moved R11 2.80 mm to (153.3, 108.5)
- moved C1 2.65 mm to (155.8, 108.5)
- moved C2 2.50 mm to (148.5, 90.5), turned to 180 degrees
- moved R8 2.02 mm to (156.8, 93.0)
- moved R6 1.50 mm to (145.0, 108.0)
- moved C10 1.50 mm to (145.0, 109.5)
- moved R7 1.03 mm to (156.8, 94.5)
- moved R1 0.90 mm to (142.0, 93.8)
- moved X1 0.50 mm to (141.0, 102.0)
- turned D1 to 180 degrees
- renumbered J20 to LED, J2 to PPM, J6 to S1, J7 to S2, J8 to S3, J9 to S4, J1 to SBUS
Connections:
- SBUS pad 1: Net-(J1-Pin_1) -> /US1RX
Routing:
- net /VDD: track 0.00 -> 76.1 mm, vias 0 -> 6
- net +5V: track 0.00 -> 31.2 mm
- net Net-(U1-VCAP_2): track 0.00 -> 16.2 mm
- net /GYRO_SDO: track 0.00 -> 14.4 mm
- net /5V_USB: track 0.00 -> 13.7 mm, vias 0 -> 2
- net /GYRO_SDA: track 0.00 -> 13.1 mm
- net Net-(U2-EN): track 0.00 -> 13.0 mm
- net /GYRO_SCL: track 0.00 -> 11.4 mm
- net Net-(SW1-B): track 0.00 -> 11.3 mm, vias 0 -> 2
- net /GYRO_CS: track 0.00 -> 10.5 mm
- net Net-(U3-REGOUT): track 0.00 -> 7.93 mm
- net Net-(U1-PC12): track 0.00 -> 6.89 mm, vias 0 -> 1
- net Net-(U1-PH1): track 0.00 -> 6.71 mm
- net /US1RX: track 0.00 -> 5.83 mm
- net Net-(Q1-B): track 0.00 -> 5.20 mm
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